File: mm_motor.kicad_sch (KiCad schematic)
At the start: 1 part, among them M1 N20_encoder

Commit message: version2
Parts:
- added C8: 2.2uF, Capacitor_SMD:C_0603_1608Metric, symbol Device:C
- added J2: Conn_01x06_Pin, symbol Connector:Conn_01x06_Pin
Connections:
- net C1: now also J2.4 (Pin_4)
- net C2: now also J2.3 (Pin_3)
- net MA: now also J2.1 (Pin_1)
- net MB: now also J2.6 (Pin_6)
- new net +BATT: C8.2, J2.5 (Pin_5)
- new net GND: C8.1, J2.2 (Pin_2)
Changed lines of the file:
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@@
 (kicad_sch (version 20230121) (generator eeschema)
   (paper "A4")
-  (hierarchical_label "C1" (shape output) (at 118.11 91.44 180) (fields_autoplaced)
-    (effects (font (size 1.27 1.27)) (justify right))
-  )
-  (hierarchical_label "C2" (shape output) (at 118.11 93.98 180) (fields_autoplaced)
-    (effects (font (size 1.27 1.27)) (justify right))
-  )
-  (hierarchical_label "MB" (shape passive) (at 118.11 99.06 180) (fields_autoplaced)
-    (effects (font (size 1.27 1.27)) (justify right))
-  )
-  (hierarchical_label "MA" (shape passive) (at 118.11 86.36 180) (fields_autoplaced)
-    (effects (font (size 1.27 1.27)) (justify right))
+  (junction (at 160.02 100.33) (diameter 0) (color 0 0 0 0)
+  )
+  (wire (pts (xy 140.97 90.17) (xy 148.59 90.17))
+    (stroke (width 0) (type default))
+  )
+  (wire (pts (xy 140.97 95.25) (xy 149.86 95.25))
+    (stroke (width 0) (type default))
+  )
+  (wire (pts (xy 140.97 97.79) (xy 149.86 97.79))
+    (stroke (width 0) (type default))
+  )
+  (wire (pts (xy 160.02 100.33) (xy 171.45 100.33))
+    (stroke (width 0) (type default))
+  )
+  (wire (pts (xy 140.97 100.33) (xy 160.02 100.33))
+    (stroke (width 0) (type default))
+  )
+  (wire (pts (xy 160.02 111.76) (xy 160.02 118.11))
+    (stroke (width 0) (type default))
+  )
+  (wire (pts (xy 160.02 104.14) (xy 160.02 100.33))
+    (stroke (width 0) (type default))
+  )
+  (wire (pts (xy 140.97 102.87) (xy 146.05 102.87))
+    (stroke (width 0) (type default))
+  )
+  (wire (pts (xy 140.97 92.71) (xy 148.59 92.71))
+    (stroke (width 0) (type default))
+  )
+  (hierarchical_label "C1" (shape output) (at 149.86 97.79 0) (fields_autoplaced)
+    (effects (font (size 1.27 1.27)) (justify left))
+  )
+  (hierarchical_label "C2" (shape output) (at 149.86 95.25 0) (fields_autoplaced)
+    (effects (font (size 1.27 1.27)) (justify left))
+  )
+  (hierarchical_label "MB" (shape passive) (at 146.05 102.87 0) (fields_autoplaced)
+    (effects (font (size 1.27 1.27)) (justify left))
+  )
+  (hierarchical_label "MA" (shape passive) (at 148.59 90.17 0) (fields_autoplaced)
+    (effects (font (size 1.27 1.27)) (justify left))
+  )
+  (symbol (lib_id "Connector:Conn_01x06_Pin") (at 135.89 95.25 0) (unit 1)
+    (in_bom yes) (on_board yes) (dnp no) (fields_autoplaced)
+    (property "Reference" "J2" (at 136.525 85.09 0)
+      (effects (font (size 1.27 1.27)))
+    )
+    (property "Value" "Conn_01x06_Pin" (at 136.525 87.63 0)
+      (effects (font (size 1.27 1.27)))
+    )
+    (property "Footprint" "" (at 135.89 95.25 0)
+      (effects (font (size 1.27 1.27)) hide)
+    )
+    (property "Datasheet" "~" (at 135.89 95.25 0)
+      (effects (font (size 1.27 1.27)) hide)
+    )
+    (pin "4")
+    (pin "2")
+    (pin "3")
+    (pin "1")
+    (pin "5")
+    (pin "6")
+    (instances
+      (project "minimouse"
+        (path "/d8fa4cba-2469-4231-847f-065b6b829f44/7f113667-692a-4f4d-b16f-621d32f3f136"
+          (reference "J2") (unit 1)
+        )
+        (path "/d8fa4cba-2469-4231-847f-065b6b829f44/3975acd0-18ad-47bc-9ce1-d8c4d864aafe"
+          (reference "J3") (unit 1)
+        )
+      )
+    )
+  )
+  (symbol (lib_id "power:+BATT") (at 171.45 100.33 270) (unit 1)
+    (in_bom yes) (on_board yes) (dnp no) (fields_autoplaced)
+    (property "Reference" "#PWR025" (at 167.64 100.33 0)
+      (effects (font (size 1.27 1.27)) hide)
+    )
+    (property "Value" "+BATT" (at 175.26 100.33 90)
+      (effects (font (size 1.27 1.27)) (justify left))
+    )
+    (property "Footprint" "" (at 171.45 100.33 0)
+      (effects (font (size 1.27 1.27)) hide)
+    )
+    (property "Datasheet" "" (at 171.45 100.33 0)
+      (effects (font (size 1.27 1.27)) hide)
+    )
+    (pin "1")
+    (instances
+      (project "minimouse"
+        (path "/d8fa4cba-2469-4231-847f-065b6b829f44/7f113667-692a-4f4d-b16f-621d32f3f136"
+          (reference "#PWR025") (unit 1)
+        )
+        (path "/d8fa4cba-2469-4231-847f-065b6b829f44/3975acd0-18ad-47bc-9ce1-d8c4d864aafe"
+          (reference "#PWR026") (unit 1)
+        )
+      )
+    )
   )
   (symbol (lib_id "minimouse:N20_w_encoder") (at 115.57 57.15 0) (unit 1)
@@
         )
       )
+    )
+  )
+  (symbol (lib_id "Device:C") (at 160.02 107.95 180) (unit 1)
+    (in_bom yes) (on_board yes) (dnp no)
+    (property "Reference" "C8" (at 153.67 107.95 90)
+      (effects (font (size 1.27 1.27)))
+    )
+    (property "Value" "2.2uF" (at 156.21 107.95 90)
+      (effects (font (size 1.27 1.27)))
+    )
+    (property "Footprint" "Capacitor_SMD:C_0603_1608Metric" (at 159.0548 104.14 0)
+      (effects (font (size 1.27 1.27)) hide)
+    )
+    (property "Datasheet" "~" (at 160.02 107.95 0)
+      (effects (font (size 1.27 1.27)) hide)
+    )
+    (pin "1")
+    (pin "2")
+    (instances
+      (project "minimouse"
+        (path "/d8fa4cba-2469-4231-847f-065b6b829f44/0999fad3-9a14-4ede-b729-a71c3dbbdf8e"
+          (reference "C8") (unit 1)
+        )
+        (path "/d8fa4cba-2469-4231-847f-065b6b829f44/7f113667-692a-4f4d-b16f-621d32f3f136"
+          (reference "C13") (unit 1)
+        )
+        (path "/d8fa4cba-2469-4231-847f-065b6b829f44/3975acd0-18ad-47bc-9ce1-d8c4d864aafe"
+          (reference "C14") (unit 1)
+        )
+      )
+    )
+  )
+  (symbol (lib_id "power:GND") (at 148.59 92.71 90) (unit 1)
+    (in_bom yes) (on_board yes) (dnp no) (fields_autoplaced)
+    (property "Reference" "#PWR027" (at 154.94 92.71 0)
+      (effects (font (size 1.27 1.27)) hide)
+    )
+    (property "Value" "GND" (at 152.4 92.71 90)
+      (effects (font (size 1.27 1.27)) (justify right))
+    )
+    (property "Footprint" "" (at 148.59 92.71 0)
+      (effects (font (size 1.27 1.27)) hide)
+    )
+    (property "Datasheet" "" (at 148.59 92.71 0)
+      (effects (font (size 1.27 1.27)) hide)
+    )
+    (pin "1")
+    (instances
+      (project "minimouse"
+        (path "/d8fa4cba-2469-4231-847f-065b6b829f44/7f113667-692a-4f4d-b16f-621d32f3f136"
+          (reference "#PWR027") (unit 1)
+        )
+        (path "/d8fa4cba-2469-4231-847f-065b6b829f44/3975acd0-18ad-47bc-9ce1-d8c4d864aafe"
+          (reference "#PWR028") (unit 1)
+        )
+      )
+    )
+  )
+  (symbol (lib_id "power:GND") (at 160.02 118.11 0) (unit 1)
+    (in_bom yes) (on_board yes) (dnp no) (fields_autoplaced)
+    (property "Reference" "#PWR029" (at 160.02 124.46 0)
+      (effects (font (size 1.27 1.27)) hide)
+    )
+    (property "Value" "GND" (at 160.02 123.19 0)
+      (effects (font (size 1.27 1.27)))
+    )
+    (property "Footprint" "" (at 160.02 118.11 0)
+      (effects (font (size 1.27 1.27)) hide)
+    )
+    (property "Datasheet" "" (at 160.02 118.11 0)
+      (effects (font (size 1.27 1.27)) hide)
+    )
+    (pin "1")
+    (instances
+      (project "minimouse"
+        (path "/d8fa4cba-2469-4231-847f-065b6b829f44/7f113667-692a-4f4d-b16f-621d32f3f136"
+          (reference "#PWR029") (unit 1)
+        )
+        (path "/d8fa4cba-2469-4231-847f-065b6b829f44/3975acd0-18ad-47bc-9ce1-d8c4d864aafe"
+          (reference "#PWR030") (unit 1)
+        )
+      )

Commit message: version 3
Parts:
- removed J2: Conn_01x06_Pin, symbol Connector:Conn_01x06_Pin
- added J7: Conn_01x06, Connector_PinHeader_2.54mm:PinHeader_1x06_P2.54mm_Vertical, symbol Connector_Generic:Conn_01x06
- added R20, R7: 100, Resistor_SMD:R_0603_1608Metric, symbol Device:R
Connections:
- net +BATT: now also J7.5 (Pin_5)
- net C1: now also R7.2
- net C2: now also R20.2
- net GND: now also J7.2 (Pin_2)
- net MA: now also J7.1 (Pin_1)
- net MB: now also J7.6 (Pin_6)
- new net: J7.3 (Pin_3), R7.1
- new net: J7.4 (Pin_4), R20.1
