File: mm_motor_control.kicad_sch (KiCad schematic)
At the start: 0 parts

Commit message: version2
Parts:
- added C10: 22nF, Capacitor_SMD:C_0603_1608Metric, symbol Device:C
- added C11, C8: 2.2uF, Capacitor_SMD:C_0603_1608Metric, symbol Device:C
- added C7: C, Capacitor_SMD:C_0603_1608Metric, symbol Device:C
- added C9: 10nF, Capacitor_SMD:C_0603_1608Metric, symbol Device:C
- added R10, R11: 330m, Resistor_SMD:R_2512_6332Metric, symbol Device:R
- added R12, R13: 18k, Resistor_SMD:R_0603_1608Metric, symbol Device:R
- added R14: 1k, Resistor_SMD:R_0603_1608Metric, symbol Device:R
- added R15: 47k, Resistor_SMD:R_0603_1608Metric, symbol Device:R
- added R16, R17: 10k, Resistor_SMD:R_0603_1608Metric, symbol Device:R
- added U2: ~, symbol minimouse:STSPIN240
Connections:
- net EN: now also R12.1
- net FAULT: now also C9.1, R12.2, U2.13 (EN/FAULT)
- net OUT_A1: now also U2.3 (OUTA1)
- net OUT_A2: now also U2.5 (OUTA2)
- net OUT_B1: now also U2.10 (OUTB1)
- net OUT_B2: now also U2.8 (OUTB2)
- net PHASE_A: now also U2.1 (PHA)
- net PHASE_B: now also U2.15 (PHB)
- net PWM_A: now also U2.2 (PWMA)
- net PWM_B: now also U2.16 (PWMB)
- net STBY/RESET: now also C7.1, R13.2, U2.14 (STBY\RESET)
- new net: R10.1, U2.4 (SENSEA)
- new net: C10.1, R14.2
- new net: R11.1, U2.9 (SENSEB)
- new net +3V3: R13.1
- new net +BATT: R17.2
- new net GND: C10.2, C11.2, C7.2, C8.2, C9.2, R10.2, R11.2, R15.2, R16.1, U2.7 (GND)
- new net REF: C11.1, R16.2, R17.1, U2.11 (REF)
- new net TOFF: R14.1, R15.1, U2.12 (TOFF)
- new net VS: C8.1, U2.6 (VS)

Commit message: version 3
Parts:
- removed C11, C8: 2.2uF, Capacitor_SMD:C_0603_1608Metric, symbol Device:C
- removed U2: ~, symbol minimouse:STSPIN240
- added U5: STSPIN240, Package_DFN_QFN:VQFN-16-1EP_3x3mm_P0.5mm_EP1.8x1.8mm, symbol Driver_Motor:STSPIN240
- C9: value 10nF -> 1nF
- R12: value 18k -> 10k
Connections:
- net +BATT: now also U5.6 (VS)
- net FAULT: now also U5.13 (EN/FLT)
- net GND: now also U5.17 (EPAD), U5.7 (GND)
- net OUT_A1: now also U5.3 (OUTA1)
- net OUT_A2: now also U5.5 (OUTA2)
- net OUT_B1: now also U5.10 (OUTB1)
- net OUT_B2: now also U5.8 (OUTB2)
- net PHASE_A: now also U5.1 (PHA)
- net PHASE_B: now also U5.15 (PHB)
- net PWM_A: now also U5.2 (PWMA)
- net PWM_B: now also U5.16 (PWMB)
- net REF: now also U5.11 (REF)
- net STBY/RESET: now also U5.14 (STBY/RESET)
- net TOFF: now also U5.12 (TOFF)
- net at R10.1: now also U5.4 (SENSEA)
- net at R11.1: now also U5.9 (SENSEB)
- net +3V3 renamed +3.3V
Other:
- moved on the sheet: C9, R10, R11, R12
