File: mm_power.kicad_sch (KiCad schematic)
At the start: 1 part, among them J5 Conn_01x02

Commit message: version2
Parts:
- added C1, C3: 1pF, Capacitor_SMD:C_0603_1608Metric, symbol Device:C
- added U3: LP5907MFX-1.2, Package_TO_SOT_SMD:SOT-23-5, symbol Regulator_Linear:LP5907MFX-1.2
Connections:
- net GND: now also C1.1, C3.1, U3.2 (GND)
- new net: C1.2, U3.1 (IN)
- new net: C3.2, U3.5 (OUT)
Changed lines of the file:
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@@
   (junction (at 86.36 82.55) (diameter 0) (color 0 0 0 0)
   )
+  (junction (at 123.19 67.31) (diameter 0) (color 0 0 0 0)
+  )
+  (junction (at 123.19 64.77) (diameter 0) (color 0 0 0 0)
+  )
+  (junction (at 152.4 64.77) (diameter 0) (color 0 0 0 0)
+  )
   (junction (at 86.36 95.25) (diameter 0) (color 0 0 0 0)
   )
+  (wire (pts (xy 118.11 64.77) (xy 123.19 64.77))
+    (stroke (width 0) (type default))
+  )
   (wire (pts (xy 86.36 90.17) (xy 86.36 95.25))
     (stroke (width 0) (type default))
   )
+  (wire (pts (xy 152.4 46.99) (xy 152.4 52.07))
+    (stroke (width 0) (type default))
+  )
   (wire (pts (xy 95.25 82.55) (xy 86.36 82.55))
     (stroke (width 0) (type default))
@@
     (stroke (width 0) (type default))
   )
+  (wire (pts (xy 152.4 64.77) (xy 160.02 64.77))
+    (stroke (width 0) (type default))
+  )
+  (wire (pts (xy 123.19 59.69) (xy 123.19 64.77))
+    (stroke (width 0) (type default))
+  )
   (wire (pts (xy 95.25 92.71) (xy 95.25 95.25))
     (stroke (width 0) (type default))
@@
     (stroke (width 0) (type default))
   )
+  (wire (pts (xy 118.11 67.31) (xy 123.19 67.31))
+    (stroke (width 0) (type default))
+  )
   (wire (pts (xy 86.36 95.25) (xy 86.36 100.33))
     (stroke (width 0) (type default))
@@
     (stroke (width 0) (type default))
   )
+  (wire (pts (xy 123.19 67.31) (xy 128.27 67.31))
+    (stroke (width 0) (type default))
+  )
   (wire (pts (xy 86.36 82.55) (xy 86.36 87.63))
     (stroke (width 0) (type default))
   )
+  (wire (pts (xy 135.89 74.93) (xy 135.89 83.82))
+    (stroke (width 0) (type default))
+  )
+  (wire (pts (xy 143.51 64.77) (xy 152.4 64.77))
+    (stroke (width 0) (type default))
+  )
+  (wire (pts (xy 123.19 67.31) (xy 123.19 71.12))
+    (stroke (width 0) (type default))
+  )
+  (wire (pts (xy 152.4 59.69) (xy 152.4 64.77))
+    (stroke (width 0) (type default))
+  )
+  (wire (pts (xy 123.19 64.77) (xy 128.27 64.77))
+    (stroke (width 0) (type default))
+  )
+  (wire (pts (xy 123.19 46.99) (xy 123.19 52.07))
+    (stroke (width 0) (type default))
+  )
   (wire (pts (xy 80.01 90.17) (xy 86.36 90.17))
     (stroke (width 0) (type default))
   )
+  (symbol (lib_id "power:GND") (at 152.4 46.99 180) (unit 1)
+    (in_bom yes) (on_board yes) (dnp no) (fields_autoplaced)
+    (property "Reference" "#PWR011" (at 152.4 40.64 0)
+      (effects (font (size 1.27 1.27)) hide)
+    )
+    (property "Value" "GND" (at 152.4 43.18 0)
+      (effects (font (size 1.27 1.27)))
+    )
+    (property "Footprint" "" (at 152.4 46.99 0)
+      (effects (font (size 1.27 1.27)) hide)
+    )
+    (property "Datasheet" "" (at 152.4 46.99 0)
+      (effects (font (size 1.27 1.27)) hide)
+    )
+    (pin "1")
+    (instances
+      (project "minimouse"
+        (path "/d8fa4cba-2469-4231-847f-065b6b829f44/3f9b0845-5778-418c-a7a8-03da2392145e"
+          (reference "#PWR011") (unit 1)
+        )
+      )
+    )
+  )
   (symbol (lib_id "power:+BATT") (at 86.36 74.93 0) (unit 1)
     (in_bom yes) (on_board yes) (dnp no) (fields_autoplaced)
@@
         (path "/d8fa4cba-2469-4231-847f-065b6b829f44/3f9b0845-5778-418c-a7a8-03da2392145e"
           (reference "#PWR036") (unit 1)
+        )
+      )
+    )
+  )
+  (symbol (lib_id "power:GND") (at 123.19 46.99 180) (unit 1)
+    (in_bom yes) (on_board yes) (dnp no) (fields_autoplaced)
+    (property "Reference" "#PWR09" (at 123.19 40.64 0)
+      (effects (font (size 1.27 1.27)) hide)
+    )
+    (property "Value" "GND" (at 123.19 43.18 0)
+      (effects (font (size 1.27 1.27)))
+    )
+    (property "Footprint" "" (at 123.19 46.99 0)
+      (effects (font (size 1.27 1.27)) hide)
+    )
+    (property "Datasheet" "" (at 123.19 46.99 0)
+      (effects (font (size 1.27 1.27)) hide)
+    )
+    (pin "1")
+    (instances
+      (project "minimouse"
+        (path "/d8fa4cba-2469-4231-847f-065b6b829f44/3f9b0845-5778-418c-a7a8-03da2392145e"
+          (reference "#PWR09") (unit 1)
+        )
+      )
+    )
+  )
+  (symbol (lib_id "Device:C") (at 123.19 55.88 0) (unit 1)
+    (in_bom yes) (on_board yes) (dnp no) (fields_autoplaced)
+    (property "Reference" "C1" (at 127 54.61 0)
+      (effects (font (size 1.27 1.27)) (justify left))
+    )
+    (property "Value" "1pF" (at 127 57.15 0)
+      (effects (font (size 1.27 1.27)) (justify left))
+    )
+    (property "Footprint" "Capacitor_SMD:C_0603_1608Metric" (at 124.1552 59.69 0)
+      (effects (font (size 1.27 1.27)) hide)
+    )
+    (property "Datasheet" "~" (at 123.19 55.88 0)
+      (effects (font (size 1.27 1.27)) hide)
+    )
+    (pin "1")
+    (pin "2")
+    (instances
+      (project "minimouse"
+        (path "/d8fa4cba-2469-4231-847f-065b6b829f44/3f9b0845-5778-418c-a7a8-03da2392145e"
+          (reference "C1") (unit 1)
         )
       )
@@
     )
   )
+  (symbol (lib_id "Device:C") (at 152.4 55.88 0) (unit 1)
+    (in_bom yes) (on_board yes) (dnp no) (fields_autoplaced)
+    (property "Reference" "C3" (at 156.21 54.61 0)
+      (effects (font (size 1.27 1.27)) (justify left))
+    )
+    (property "Value" "1pF" (at 156.21 57.15 0)
+      (effects (font (size 1.27 1.27)) (justify left))
+    )
+    (property "Footprint" "Capacitor_SMD:C_0603_1608Metric" (at 153.3652 59.69 0)
+      (effects (font (size 1.27 1.27)) hide)
+    )
+    (property "Datasheet" "~" (at 152.4 55.88 0)
+      (effects (font (size 1.27 1.27)) hide)
+    )
+    (pin "1")
+    (pin "2")
+    (instances
+      (project "minimouse"
+        (path "/d8fa4cba-2469-4231-847f-065b6b829f44/3f9b0845-5778-418c-a7a8-03da2392145e"
+          (reference "C3") (unit 1)
+        )
+      )
+    )
+  )
+  (symbol (lib_id "Regulator_Linear:LP5907MFX-1.2") (at 135.89 67.31 0) (unit 1)
+    (in_bom yes) (on_board yes) (dnp no) (fields_autoplaced)
+    (property "Reference" "U3" (at 135.89 57.15 0)
+      (effects (font (size 1.27 1.27)))
+    )
+    (property "Value" "LP5907MFX-1.2" (at 135.89 59.69 0)
+      (effects (font (size 1.27 1.27)))
+    )
+    (property "Footprint" "Package_TO_SOT_SMD:SOT-23-5" (at 135.89 58.42 0)
+      (effects (font (size 1.27 1.27)) hide)
+    )
+    (property "Datasheet" "http://www.ti.com/lit/ds/symlink/lp5907.pdf" (at 135.89 54.61 0)
+      (effects (font (size 1.27 1.27)) hide)
+    )
+    (pin "2")
+    (pin "4")
+    (pin "3")
+    (pin "1")
+    (pin "5")
+    (instances
+      (project "minimouse"
+        (path "/d8fa4cba-2469-4231-847f-065b6b829f44/3f9b0845-5778-418c-a7a8-03da2392145e"
+          (reference "U3") (unit 1)
+        )
+      )
+    )
+  )
   (symbol (lib_id "Connector_Generic:Conn_01x02") (at 74.93 90.17 180) (unit 1)
     (in_bom yes) (on_board yes) (dnp no) (fields_autoplaced)
@@
         )
       )
+    )
+  )
+  (symbol (lib_id "power:GND") (at 135.89 83.82 0) (unit 1)
+    (in_bom yes) (on_board yes) (dnp no) (fields_autoplaced)
+    (property "Reference" "#PWR08" (at 135.89 90.17 0)
+      (effects (font (size 1.27 1.27)) hide)
+    )
+    (property "Value" "GND" (at 135.89 88.9 0)
+      (effects (font (size 1.27 1.27)))
+    )
+    (property "Footprint" "" (at 135.89 83.82 0)
+      (effects (font (size 1.27 1.27)) hide)
+    )
+    (property "Datasheet" "" (at 135.89 83.82 0)
+      (effects (font (size 1.27 1.27)) hide)
+    )
+    (pin "1")
+    (instances
+      (project "minimouse"
+        (path "/d8fa4cba-2469-4231-847f-065b6b829f44/3f9b0845-5778-418c-a7a8-03da2392145e"
+          (reference "#PWR08") (unit 1)
+        )
+      )

Commit message: version 3
Parts:
- added D1: LED, LED_SMD:LED_0603_1608Metric, symbol Device:LED
- added R18: 330, Resistor_SMD:R_0603_1608Metric, symbol Device:R
- C20: renamed from C3; value 1pF -> 2.2uF
- C21: renamed from C1; value 1pF -> 2.2uF
Connections:
- net +BATT: now also C21.1, U3.1 (IN), U3.3 (EN)
- net GND: now also C20.2, C21.2, D1.1 (K); no longer C20.1, C21.1
- net +3.3V: now reaches U3.5 (OUT)
- net +3.3V: now also C20.1, R18.1; no longer C20.2
- new net: D1.2 (A), R18.2
Other:
- moved on the sheet: C20, C21, J5
