File: minimouse.kicad_pcb (KiCad board)
At the start: 2 copper layers, 90 x 85 mm, 22 parts, among them J1 Conn_ARM_JTAG_SWD_10, J5 Conn_01x02, M1 N20_encoder, M2 N20_encoder, U1 STM32F030C8Tx, U4 HC-SR04

Commit message: version4
Parts:
- added C10: 22nF, Capacitor_SMD:C_0603_1608Metric, F.Cu at (167.1, 92.6)
- added C11: 2.2uF, Capacitor_SMD:C_0603_1608Metric, F.Cu at (85.6, 78.5)
- added C12: 2.2uF, Capacitor_SMD:C_0603_1608Metric, F.Cu at (177.9, 72.8)
- added C13: 2.2uF, Capacitor_SMD:C_0603_1608Metric, F.Cu at (85.6, 83.6)
- added C20: 2.2uF, Capacitor_SMD:C_0603_1608Metric, F.Cu at (140.6, 100.5)
- added C21: 2.2uF, Capacitor_SMD:C_0603_1608Metric, F.Cu at (85.6, 81.1)
- added C7: C, Capacitor_SMD:C_0603_1608Metric, F.Cu at (173.8, 95.2)
- added C8: 2.2uF, Capacitor_SMD:C_0603_1608Metric, F.Cu at (85.6, 86.1)
- added C9: 1nF, Capacitor_SMD:C_0603_1608Metric, F.Cu at (215.3, 65.4)
- added D1: LED, LED_SMD:LED_0603_1608Metric, F.Cu at (143.4, 104.3)
- added J4: Conn_01x04_Pin, Connector_PinHeader_2.54mm:PinHeader_1x04_P2.54mm_Vertical, F.Cu at (125.5, 94.9)
- added J6: Conn_01x06, Connector_PinHeader_2.54mm:PinHeader_1x06_P2.54mm_Vertical, F.Cu at (166.6, 106.5)
- added J7: Conn_01x06, Connector_PinHeader_2.54mm:PinHeader_1x06_P2.54mm_Vertical, F.Cu at (92.2, 75.5)
- added R10: 330m, Resistor_SMD:R_2512_6332Metric, F.Cu at (180.1, 89.8)
- added R11: 330m, Resistor_SMD:R_2512_6332Metric, F.Cu at (167.9, 86.7)
- added R12: 10k, Resistor_SMD:R_0603_1608Metric, F.Cu at (230.5, 92.4)
- added R13: 18k, Resistor_SMD:R_0603_1608Metric, F.Cu at (175.5, 95.2)
- added R14: 1k, Resistor_SMD:R_0603_1608Metric, F.Cu at (170.2, 92.6)
- added R15: 47k, Resistor_SMD:R_0603_1608Metric, F.Cu at (170.2, 94.2)
- added R16: 10k, Resistor_SMD:R_0603_1608Metric, F.Cu at (170.2, 91.0)
- added R17: 10k, Resistor_SMD:R_0603_1608Metric, F.Cu at (170.2, 89.5)
- added R18: 330, Resistor_SMD:R_0603_1608Metric, F.Cu at (143.4, 101.2)
- added R19: 100, Resistor_SMD:R_0603_1608Metric, F.Cu at (234.7, 65.4)
- added R20: 100, Resistor_SMD:R_0603_1608Metric, F.Cu at (245.3, 65.4)
- added R21: 100, Resistor_SMD:R_0603_1608Metric, F.Cu at (234.7, 67.9)
- added R22: 100, Resistor_SMD:R_0603_1608Metric, F.Cu at (130.7, 83.2)
- added U3: LP5907MFX-1.2, Package_TO_SOT_SMD:SOT-23-5, F.Cu at (140.8, 103.5)
- added U5: STSPIN240, Package_DFN_QFN:VQFN-16-1EP_3x3mm_P0.5mm_EP1.8x1.8mm, F.Cu at (174.0, 91.5)
- moved R1 82.3 mm to (216.3, 33.0)
- moved R9 82.3 mm to (213.9, 33.1)
- moved BOOT0 78.3 mm to (221.9, 34.2)
- moved R6 53.0 mm to (98.2, 107.9)
- moved J1 51.0 mm to (214.9, 82.6)
- moved R3 49.6 mm to (93.5, 97.6)
- moved C5 46.7 mm to (167.8, 72.8), turned to -90 degrees
- moved R2 45.4 mm to (98.0, 85.5), turned to 90 degrees
- moved R4 39.7 mm to (104.9, 101.9)
- moved C6 33.4 mm to (175.4, 72.8), turned to -90 degrees
- moved C3 31.1 mm to (170.3, 72.8), turned to -90 degrees
- moved C2 29.5 mm to (172.9, 72.8), turned to -90 degrees
- moved C1 29.2 mm to (165.2, 72.8), turned to -90 degrees
- moved R7 28.2 mm to (124.6, 105.9)
- moved R5 27.3 mm to (119.5, 105.9)
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Connections:
- R6 pad 1: /mcu/OUT_B0 -> /motor_control/STBY\RESET
- R7 pad 1: /mcu/OUT_B1 -> Net-(J6-Pin_3)
- R7 pad 2: Net-(U1-PB1) -> /mcu/TIM3_CH1
- R8 pad 1: /mcu/UART1_TX -> /external_uart/EXT_UART_RX
- U1 pad 19: Net-(U1-PB1) -> /mcu/OUT_B1
- U1 pad 43: /mcu/UART1_RX -> /external_uart/EXT_UART_TX
- U4 pad 3: Net-(U4-ECHO) -> /mcu/TIM8_CH2
- U4 pad 4: +3V3 -> +3.3V

Commit message: version4
Parts:
- moved R19 110.9 mm to (129.4, 100.3), turned to 90 degrees
- moved R21 107.6 mm to (132.1, 100.3), turned to 90 degrees
- moved R20 91.3 mm to (160.9, 100.1), turned to 90 degrees
- moved R12 89.1 mm to (141.4, 93.2), turned to -90 degrees
- moved C21 89.0 mm to (172.2, 101.4), turned to -90 degrees
- moved BOOT0 81.4 mm to (151.2, 74.7)
- moved R1 79.1 mm to (148.8, 74.3)
- moved R9 78.6 mm to (147.0, 74.3)
- moved C9 77.4 mm to (143.1, 93.2), turned to 90 degrees
- moved C8 73.8 mm to (158.0, 100.3), turned to -90 degrees
- moved R6 56.1 mm to (150.6, 87.9)
- moved C11 53.6 mm to (134.5, 100.4), turned to -90 degrees
- moved R3 52.6 mm to (144.9, 86.4)
- moved J1 47.6 mm to (168.3, 73.1), turned to -90 degrees
- moved R2 44.9 mm to (142.9, 85.0), turned to -90 degrees
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
Commit message: version6
Parts:
- moved J4 46.9 mm to (168.7, 81.3)
- moved C13 40.0 mm to (165.2, 83.6), turned to 0 degrees
- moved R22 39.8 mm to (165.0, 86.3), turned to 180 degrees
- moved C6 23.0 mm to (156.2, 89.7), turned to 0 degrees
- moved R13 16.1 mm to (154.6, 96.4)
- moved R12 15.9 mm to (153.8, 103.2)
- moved C9 15.9 mm to (153.0, 105.6), turned to 180 degrees
- moved R17 15.8 mm to (155.9, 109.5)
- moved R16 15.7 mm to (155.9, 107.9)
- moved R15 15.1 mm to (157.2, 104.3)
- moved U5 14.8 mm to (150.0, 109.8)
- moved C10 14.7 mm to (159.9, 102.8)
- moved R14 14.7 mm to (157.2, 102.1)
- moved R11 14.5 mm to (158.1, 113.7), turned to 0 degrees
- moved C7 14.1 mm to (151.5, 102.2)
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
Commit message: version7
Parts:
- moved C6 16.6 mm to (141.9, 81.4), turned to 90 degrees
- moved BOOT0 6.06 mm to (152.4, 72.5)
- moved C1 4.83 mm to (170.7, 72.3)
- moved R13 3.89 mm to (150.7, 96.8), turned to 0 degrees
- moved C4 3.60 mm to (157.6, 90.4)
- moved R5 2.29 mm to (149.1, 92.9)
- moved C3 1.87 mm to (144.1, 84.5)
- moved C2 1.17 mm to (144.2, 81.3)
- moved J6 1.06 mm to (178.7, 104.2)
- moved R6 0.97 mm to (150.8, 93.0)
- moved C21 0.94 mm to (181.1, 93.8)
- moved R11 0.69 mm to (157.5, 114.0)
- moved C11 0.64 mm to (131.1, 99.6)
- moved R19 0.64 mm to (126.0, 99.5)
- moved R21 0.64 mm to (128.7, 99.5)
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Routing:
- net +BATT: track 0.00 -> 196.7 mm
- net +3.3V: track 0.00 -> 145.6 mm
- net /motorB/MB: track 0.00 -> 32.1 mm
- net /motorA/MB: track 0.00 -> 28.3 mm
- net /mcu/TIM2_CH1: track 0.00 -> 25.7 mm
- net /mcu/IN_B2: track 0.00 -> 23.2 mm
- net /mcu/TIM2_CH2: track 0.00 -> 22.8 mm
- net /mcu/SWDIO: track 0.00 -> 17.1 mm
- net /mcu/SWO: track 0.00 -> 16.4 mm
- net /mcu/SWDCLK: track 0.00 -> 16.2 mm
- net /mcu/TIM15_CH1: track 0.00 -> 15.9 mm
- net /mcu/OUT_A4: track 0.00 -> 15.6 mm
- net /mcu/OUT_A5: track 0.00 -> 14.8 mm
- net /mcu/OUT_B1: track 0.00 -> 14.2 mm
- net /mcu/TIM8_CH2: track 0.00 -> 12.5 mm
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
Commit message: final
Parts:
- added R23: 100, Resistor_SMD:R_0603_1608Metric, F.Cu at (150.1, 72.4)
- moved J6 12.8 mm to (165.9, 104.1), turned to 90 degrees
- moved C12 11.9 mm to (168.0, 70.8)
- moved C8 6.99 mm to (176.1, 100.3)
- moved R9 4.69 mm to (148.7, 77.7)
- moved R10 3.76 mm to (142.8, 111.1)
- moved R7 3.63 mm to (170.9, 100.7)
- moved R11 3.01 mm to (157.7, 111.0)
- moved R16 2.32 mm to (157.3, 106.0)
- moved R17 2.32 mm to (157.3, 107.7)
- moved C5 1.53 mm to (145.3, 78.6)
- moved R20 1.49 mm to (173.4, 100.8)
Connections:
- U4 pad 3: /mcu/TIM8_CH2 -> Net-(U4-ECHO)
- U4 pad 4: +3.3V -> +BATT
Routing:
- net +BATT: track 196.7 -> 249.4 mm
- net /motorB/MA: track 0.00 -> 32.6 mm, vias 0 -> 2
- net /mcu/TIM3_CH2: track 0.00 -> 30.5 mm, vias 0 -> 2
- net /mcu/TIM3_CH1: track 0.00 -> 26.5 mm, vias 0 -> 2
- net /mcu/~{RESET}: track 0.00 -> 26.1 mm, vias 0 -> 2
- net +3.3V: track 145.6 -> 124.2 mm, vias 0 -> 3
- net /external_uart/EXT_UART_RX: track 0.00 -> 21.2 mm, vias 0 -> 2
- net /motorA/MA: track 0.00 -> 17.6 mm
- net /external_uart/EXT_UART_TX: track 0.00 -> 16.3 mm, vias 0 -> 2
- net /motorA/MB: track 28.3 -> 44.3 mm
- net /motor_control/STBY\RESET: track 7.84 -> 15.5 mm
- net /motor_control/TOFF: track 2.24 -> 9.33 mm
- net /mcu/OUT_B9: track 3.23 -> 8.28 mm
- net Net-(U1-PB9): track 7.40 -> 2.59 mm
- net /mcu/TIM8_CH2: track 12.5 -> 7.89 mm
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- added copper zone on B.Cu, net GND

Commit message: final
Parts:
- moved J7 14.8 mm to (135.7, 103.7), turned to -90 degrees
- moved R2 9.38 mm to (144.6, 89.8)
- moved C11 5.37 mm to (125.7, 99.2)
- moved R19 4.95 mm to (130.9, 99.7)
- moved R21 0.64 mm to (128.2, 100.0)
- moved R10 0.47 mm to (142.3, 111.0)
Connections:
- U1 pad 10: /mcu/TIM2_CH1 -> /mcu/TIM2_CH2
- U1 pad 11: /mcu/TIM2_CH2 -> /mcu/TIM2_CH1
Routing:
- net +BATT: track 249.4 -> 284.6 mm
- net /motorB/MA: track 32.6 -> 15.4 mm, vias 2 -> 0
- net Net-(U1-PA2): track 11.8 -> 2.61 mm
- net /mcu/TIM2_CH1: track 25.7 -> 20.6 mm
- net /motorB/MB: track 32.5 -> 37.5 mm
- net /mcu/TIM15_CH1: track 15.9 -> 20.7 mm
- net /mcu/TIM2_CH2: track 22.8 -> 23.6 mm
