File: mm_mcu.kicad_sch (KiCad schematic)
At the start: 17 parts, among them J1 Conn_ARM_JTAG_SWD_10, U1 STM32F030C8Tx

Commit message: final
Connections:
- net TIM2_CH1: now also U1.11 (PA1); no longer U1.10 (PA0)
- net TIM2_CH2: now also U1.10 (PA0); no longer U1.11 (PA1)
